Commit message: Point body in the right direction.

File: urdf/no_stl_drone.urdf.xacro (robot description, xacro)
@@ -1,6 +1,6 @@
 <?xml version="1.0"?>
 <robot xmlns:xacro="http://www.ros.org/wiki/xacro" name="ardrone">
-  <xacro:property name="base_length" value="0.43"/>
-  <xacro:property name="base_width" value="0.07"/>
+  <xacro:property name="base_width" value="0.43"/>
+  <xacro:property name="base_length" value="0.07"/>
   <xacro:property name="base_height" value="0.04"/>
   <xacro:property name="hull_radius" value="0.125"/>

Commit message: Simplify hull_circle definition by removing block.

File: urdf/no_stl_drone.urdf.xacro (robot description, xacro)
@@ -6,5 +6,5 @@
   <xacro:property name="hull_radius" value="0.125"/>
   <xacro:property name="hull_height" value="0.02"/>
-  <xacro:macro name="hull_circle" params="name x y material *colour">
+  <xacro:macro name="hull_circle" params="name x y material rgba">
     <link name="${name}">
       <visual>
@@ -13,5 +13,5 @@
 	</geometry>
 	<material name="${material}">
-	  <xacro:insert_block name="colour"/>
+	  <color rgba="${rgba}"/>
 	</material>
       </visual>
@@ -30,15 +30,7 @@
     </visual>
   </link>
-  <xacro:hull_circle name="front_left" x="-1" y="1" material="white">
-    <color rgba="1 1 1 1"/>
-  </xacro:hull_circle>
-  <xacro:hull_circle name="front_right" x="1" y="1" material="white">
-    <color rgba="1 1 1 1"/>
-  </xacro:hull_circle>
-  <xacro:hull_circle name="aft_left" x="-1" y="-1" material="blue">
-    <color rgba="0 0 0.8 1"/>
-  </xacro:hull_circle>
-  <xacro:hull_circle name="aft_right" x="1" y="-1" material="blue">
-    <color rgba="0 0 0.8 1"/>
-  </xacro:hull_circle>
+  <xacro:hull_circle name="front_left" x="-1" y="1" material="white" rgba="1 1 1 1"/>
+  <xacro:hull_circle name="front_right" x="1" y="1" material="white" rgba="1 1 1 1"/>
+  <xacro:hull_circle name="aft_left" x="-1" y="-1" material="blue" rgba="0 0 0.8 1"/>
+  <xacro:hull_circle name="aft_right" x="1" y="-1" material="blue" rgba="0 0 0.8 1"/>
 </robot>
