Commit message: Add urdf file for drone.

File: urdf/no_stl_drone.urdf (robot description, URDF)
Before this commit: robot ardrone, 5 links, 4 joints
Links:
- link base_link: geometry visual box size=0.07 0.43 0.04
Joints:
- joint base_to_aft_left: origin xyz=0.125 -0.125 0 -> xyz=-0.125 -0.125 0
- joint base_to_aft_right: origin xyz=0.125 0.125 0 -> xyz=0.125 -0.125 0
- joint base_to_front_left: origin xyz=-0.125 -0.125 0 -> xyz=-0.125 0.125 0
- joint base_to_front_right: origin xyz=-0.125 0.125 0 -> xyz=0.125 0.125 0
