Commit message: Rename base_link to ardrone/base_link to be able to display in rviz.

File: urdf/drone.urdf (robot description, URDF)
Before this commit: robot ardrone, 1 links, 0 joints
Links:
- removed link base_link
- added link ardrone/base_link; visual mesh filename=package://spirit/meshes/drone_small.dae

Commit message: Rename ardrone/base_link to ardrone/body

File: urdf/drone.urdf (robot description, URDF)
Before this commit: robot ardrone, 1 links, 0 joints
Links:
- removed link ardrone/base_link
- added link ardrone/body; visual mesh filename=package://spirit/meshes/drone_small.dae

File: urdf/no_stl_drone.urdf (robot description, URDF)
Before this commit: robot ardrone, 5 links, 4 joints
Links:
- removed link base_link
- added link body; visual box size=0.07 0.43 0.04
Joints:
- joint base_to_aft_left: parent base_link -> body
- joint base_to_aft_right: parent base_link -> body
- joint base_to_front_left: parent base_link -> body
- joint base_to_front_right: parent base_link -> body

File: urdf/no_stl_drone.urdf.xacro (robot description, xacro)
@@ -18,10 +18,10 @@
     </link>
     <joint name="base_to_${name}" type="fixed">
-      <parent link="base_link"/>
+      <parent link="body"/>
       <child link="${name}"/>
       <origin xyz="${hull_radius*x} ${hull_radius*y} 0"/>
     </joint>
   </xacro:macro>
-  <link name="base_link">
+  <link name="body">
     <visual>
       <geometry>
