Commit message: Open drone control and joystick as necessary.

File: launch/xacro/camera.launch.xacro (robot description, xacro)
@@ -28,14 +28,4 @@
         </node>
     </xacro:macro>
-    <xacro:macro name="tum_gui" >
-        <node name="drone_autopilot"
-              pkg="tum_ardrone"
-              type="drone_autopilot"
-              output="screen" />
-        <node name="drone_gui"
-              pkg="tum_ardrone"
-              type="drone_gui"
-              output="screen" />
-    </xacro:macro>
     <xacro:if value="${params['camera']['mock_camera']}">
         <xacro:mock_camera />
@@ -43,7 +33,4 @@
     <xacro:unless value="${params['camera']['mock_camera']}">
         <xacro:ardrone_camera />
-        <xacro:if value="${params['camera']['real']['use_tum']}">
-            <xacro:tum_gui />
-        </xacro:if>
     </xacro:unless>
     <node name="reduce_framerate" pkg="spirit" type="reduce_framerate.py" output="screen">

Commit message: Automatically generate drone ip and joystick number.

File: launch/xacro/camera.launch.xacro (robot description, xacro)
@@ -1,5 +1,5 @@
 <?xml version="1.0"?>
 <launch xmlns:xacro="http://www.ros.org/wiki/xacro">
-    <xacro:property name="params" value="${load_yaml('../../config/launch_params.yaml')}"/>
+    <xacro:property name="params" value="${load_yaml('../../config/.launch_params.yaml')}"/>
     <xacro:macro name="ardrone_camera" >
         <node name="ardrone"

File: launch/xacro/control.launch.xacro (robot description, xacro)
@@ -1,5 +1,5 @@
 <?xml version="1.0"?>
 <launch xmlns:xacro="http://www.ros.org/wiki/xacro">
-    <xacro:property name="params" value="${load_yaml('../../config/launch_params.yaml')}"/>
+    <xacro:property name="params" value="${load_yaml('../../config/.launch_params.yaml')}"/>
     <xacro:macro name="joystick_gui" >
     <rosparam param="joy_node/dev">

File: launch/xacro/display.launch.xacro (robot description, xacro)
@@ -1,5 +1,5 @@
 <?xml version="1.0"?>
 <launch xmlns:xacro="http://www.ros.org/wiki/xacro">
-    <xacro:property name="params" value="${load_yaml('../../config/launch_params.yaml')}"/>
+    <xacro:property name="params" value="${load_yaml('../../config/.launch_params.yaml')}"/>
     <xacro:macro name="display" params="topic title">
         <node name="display_${topic}" pkg="spirit" type="display_video.py" output="screen">

File: launch/xacro/past_images.launch.xacro (robot description, xacro)
@@ -2,5 +2,5 @@
 <!--Generated automatically from launch config file.-->
 <launch xmlns:xacro="http://www.ros.org/wiki/xacro">
-  <xacro:property name="params" value="${load_yaml('../../config/launch_params.yaml')}"/>
+  <xacro:property name="params" value="${load_yaml('../../config/.launch_params.yaml')}"/>
   <xacro:property name="method" value="${params['past_image']['general']['eval_method']}"/>
   <xacro:property name="method_ns" value="${params['past_image'][method]}"/>

File: launch/xacro/pose.launch.xacro (robot description, xacro)
@@ -1,5 +1,5 @@
 <?xml version="1.0"?>
 <launch xmlns:xacro="http://www.ros.org/wiki/xacro">
-    <xacro:property name="params" value="${load_yaml('../../config/launch_params.yaml')}" />
+    <xacro:property name="params" value="${load_yaml('../../config/.launch_params.yaml')}" />
     <xacro:property name="real" value="${params['pose']['real']}" />
     <xacro:macro name="mocap">

File: launch/xacro/visualization.launch.xacro (robot description, xacro)
@@ -1,5 +1,5 @@
 <?xml version="1.0"?>
 <launch xmlns:xacro="http://www.ros.org/wiki/xacro">
-    <xacro:property name="params" value="${load_yaml('../../config/launch_params.yaml')}"/>
+    <xacro:property name="params" value="${load_yaml('../../config/.launch_params.yaml')}"/>
     <xacro:if value="${params['visualization']['show']}">
       <node name="visualizer" pkg="spirit" type="visualizer.py" output="screen">

Commit message: Incorporate ardrone_tutorial.

File: launch/xacro/camera.launch.xacro (robot description, xacro)
@@ -2,14 +2,22 @@
 <launch xmlns:xacro="http://www.ros.org/wiki/xacro">
     <xacro:property name="params" value="${load_yaml('../../config/.launch_params.yaml')}"/>
-    <xacro:macro name="ardrone_camera" >
+    <xacro:macro name="ardrone_driver" >
         <node name="ardrone"
               pkg="ardrone_autonomy"
               type="ardrone_driver"
               output="screen"
+              clear_params="true"
               args="-ip ${params['camera']['real']['drone_ip']}" >
             <param name="navdata_demo" value="False" />
             <param name="realtime_navdata" value="True" />
             <param name="realtime_video" value="True" />
-            <param name="looprate" value="30" />
+            <param name="looprate" value="200" />
+            <param name="outdoor" value="0" />
+            <param name="flight_without_shell" value="0" />
+            <param name="altitude_max" value="2000" />  <!-- in millimeters -->
+            <param name="altitude_min" value="50" />  <!-- in millimeters -->
+            <param name="euler_angle_max" value="0.1" />  <!-- maximum allowable body angle in radians = 5 degrees -->
+            <param name="control_vz_max" value="200" />  <!-- maximum z velocity in mm/sec = 0.2 m/sec -->
+            <param name="control_yaw" value="0.7" />  <!-- maximum rotation rate in radians/sec = 40 deg per second -->
         </node>
     </xacro:macro>
@@ -32,5 +40,5 @@
     </xacro:if>
     <xacro:unless value="${params['camera']['mock_camera']}">
-        <xacro:ardrone_camera />
+        <xacro:ardrone_driver />
     </xacro:unless>
     <node name="reduce_framerate" pkg="spirit" type="reduce_framerate.py" output="screen">

File: launch/xacro/control.launch.xacro (robot description, xacro)
@@ -3,22 +3,35 @@
     <xacro:property name="params" value="${load_yaml('../../config/.launch_params.yaml')}"/>
     <xacro:macro name="joystick_gui" >
-    <rosparam param="joy_node/dev">
-        /dev/input/js${params['control']['js_number']}
-    </rosparam>
-        <node name="drone_autopilot"
-              pkg="tum_ardrone"
-              type="drone_autopilot"
-              output="screen" />
-        <node name="drone_gui"
-              pkg="tum_ardrone"
-              type="drone_gui"
-              output="screen" />
-    <node name="joy_node"
-          pkg="joy"
-          type="joy_node"
-          output="screen" />
+        <node name="joy_node"
+              pkg="joy"
+              type="joy_node"
+              output="screen"
+              clear_params="true" >
+            <param name="dev" type="str" value="/dev/input/js${params['control']['js_number']}" />
+        </node>
+        <!-- Launches the joystick controller -->
+	    <node name="joystick_controller"
+              pkg="ardrone_tutorials"
+              type="joystick_controller.py"
+              output="screen"
+              required="true">
+            <!-- Configures the joystick button mapping -->
+            <param name="ButtonEmergency" value="11" />
+            <param name="ButtonLand" value="8" />
+            <param name="ButtonTakeoff" value="10" />
+            <!-- Configures the joystick axis mapping -->
+            <param name="AxisRoll" value="0" />
+            <param name="AxisPitch" value="1" />
+            <param name="AxisYaw" value="2" />
+            <param name="AxisZ"	value="3" />
+            <!-- Configures the joystick mapping -->
+            <param name="ScaleRoll" value="1" />
+            <param name="ScalePitch" value="1" />
+            <param name="ScaleYaw" value="1" />
+            <param name="ScaleZ" value="1" />
+	    </node>
     </xacro:macro>
     <xacro:if value="${params['control']['use_joystick']}">
-      <xacro:joystick_gui />
+        <xacro:joystick_gui />
     </xacro:if>
 </launch>
